File: pwmfan.sch (KiCad schematic (older format))
At the start: 32 parts, among them J1 Conn_ARM_JTAG_SWD_10, J2 PWR_IN, M1 Fan_4pin, Q1 Q_NMOS_DGS, SW1 SW_Push, SW2 SW_Push, U2 STM32F042F6Px, U3 NCP1117-3.3_SOT223

Commit message: Various tweaks and adding more LEDs
Parts:
- removed R1, R2, R3, R4: 680r, Resistor_SMD:R_0603_1608Metric, symbol Device:R_Small
- removed R10, R9: 10k, Resistor_SMD:R_0603_1608Metric, symbol Device:R_Small
- removed SW1, SW2: SW_Push, Button_Switch_THT:SW_Tactile_SPST_Angled_PTS645Vx83-2LFS, symbol Switch:SW_Push
- added D5, D6, D7, D8: LED_Small, LED_THT:LED_D3.0mm_Horizontal_O1.27mm_Z2.0mm, symbol Device:LED_Small
- added IC1: NPIC6C596A, Package_SO:TSSOP-16_4.4x5mm_P0.65mm, symbol agg-kicad:NPIC6C596A
- added R11, R12: 10k, Resistor_SMD:R_0603_1608Metric, symbol Device:R_Small
- added RN1, RN2: 680r, Resistor_SMD:R_Array_Convex_4x0612, symbol Device:R_Pack04
- SW1: renamed from SW?; value Rotary_Encoder -> RE111F-20B; footprint (none) -> pwmfan:RE111F-20B
Connections:
- net SW_UP is gone; now on net ENC_A: U2.11 (PA5)
- net +3V3: now also SW1.C, D5.2 (A), D6.2 (A), D7.2 (A), D8.2 (A), IC1.1 (VCC), IC1.7 (~MR)
- net GND: now also IC1.16 (GND), IC1.8 (~OE), R11.2, R12.2
- net PWM: now also U2.13 (PA7); no longer U2.12 (PA6)
- net at D2.1 (K): now also RN1.2 (R2.1)
- net at D3.1 (K): now also RN1.3 (R3.1)
- net at D4.1 (K): now also RN1.4 (R4.1)
- net SHIFT_CLK: now reaches U2.8 (PA2)
- net SHIFT_CLK: now also IC1.15 (SHCP)
- net SERIAL: now reaches U2.6 (PA0)
- net SERIAL: now also IC1.2 (DS)
- net STORE_CLK: now reaches U2.7 (PA1)
- net STORE_CLK: now also IC1.10 (STCP)
- net at D1.1 (K): now also RN1.1 (R1.1)
- net ENC_A: now reaches SW1.A
- net ENC_A: now also R11.1
- net ENC_B: now reaches SW1.B
- net ENC_B: now also U2.12 (PA6), R12.1
- net SW_DOWN: no longer names the net of U2.10 (PA4)
- new net: IC1.11 (Q4), RN2.4 (R4.1)
- new net: IC1.12 (Q5), RN2.3 (R3.1)
- new net: IC1.13 (Q6), RN2.2 (R2.1)
- new net: IC1.14 (Q7), RN2.1 (R1.1)
- new net: IC1.3 (Q0), RN1.8 (R1.2)
- new net: IC1.4 (Q1), RN1.7 (R2.2)
- new net: IC1.5 (Q2), RN1.6 (R3.2)
- new net: IC1.6 (Q3), RN1.5 (R4.2)
- new net: D7.1 (K), RN2.7 (R2.2)
- new net: D6.1 (K), RN2.6 (R3.2)
- new net: D5.1 (K), RN2.5 (R4.2)
- new net: D8.1 (K), RN2.8 (R1.2)
- no-connect marks 8 -> 15
Other:
- note added: "Display"
- moved on the sheet: C6, C7, D1, D2, D3, D4, D9, F1, H1, H2, J1, J2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
