File: pwmfan.sch (KiCad schematic (older format))
At the start: 33 parts, among them IC1 NPIC6C596A, J1 Conn_ARM_JTAG_SWD_10, J2 PWR_IN, M1 Fan_4pin, Q1 Q_NMOS_DGS, SW1 RE111F-20B, U2 STM32F042F6Px, U3 NCP1117-3.3_SOT223

Commit message: Various updates and silks
Parts:
- removed D9: TS4148RXG, Diode_SMD:D_1206_3216Metric, symbol Device:D_Small
- added Q2: DMG2307L, Package_TO_SOT_SMD:SOT-23, symbol Device:Q_PMOS_GSD
- added R1, R2: 10k, Resistor_SMD:R_0603_1608Metric, symbol Device:R_Small
- added R3: 3k3, Resistor_SMD:R_0603_1608Metric, symbol Device:R_Small
- added R4: PIN, Resistor_SMD:R_0603_1608Metric, symbol Device:R_Small
- added SYM1: QR, pwmfan:QR, symbol Graphic:SYM_Hot_Small
- Q1: value Q_NMOS_DGS -> BSS316N; symbol Device:Q_NMOS_DGS -> Device:Q_NMOS_GSD; Farnell (none) -> 2432720
- R5: value 0r -> BRD
- R6: value 100k -> 10k
- U3: value NCP1117-3.3_SOT223 -> NCP1117-3.3
Connections:
- net +12V: now also Q2.2 (S), R2.1; no longer F1.1
- net +3V3: now also R6.1
- net GND: now also Q1.2 (S), Q2.1 (G), R3.2; no longer Q1.3 (S), R6.2
- net PWM: now also R4.1
- net at Q1.1 (G): now also R5.1, R6.2; no longer M1.1 (-)
- net TACHO: now reaches U2.14 (PB1)
- net TACHO: now also R1.2, R3.1
- net at M1.3 (Tacho): now also R1.1, R2.2
- net at M1.4 (PWM): now also R4.2
- new net: M1.1 (-), Q1.3 (D)
- new net: F1.1, Q2.3 (D)
- no-connect marks 15 -> 12
Other:
- moved on the sheet: C6, C7, F1, J1, J2, M1, R11, R12, R5, R6, SW1, U3

Commit message: Minor tweaks before shipping
Parts:
- RN1, RN2: value 680r -> 4x680r
Changed lines of the file:
@@
 P 5600 1300
 F 0 "RN1" H 5320 1254 50  0000 R CNN
-F 1 "680r" H 5320 1345 50  0000 R CNN
+F 1 "4x680r" H 5320 1345 50  0000 R CNN
 F 2 "Resistor_SMD:R_Array_Convex_4x0612" V 5875 1300 50  0001 C CNN
 F 3 "~" H 5600 1300 50  0001 C CNN
@@
 P 5900 1300
 F 0 "RN2" H 5620 1346 50  0000 R CNN
-F 1 "680r" H 5620 1255 50  0000 R CNN
+F 1 "4x680r" H 5620 1255 50  0000 R CNN
 F 2 "Resistor_SMD:R_Array_Convex_4x0612" V 6175 1300 50  0001 C CNN
 F 3 "~" H 5900 1300 50  0001 C CNN
