File: pwmfan.kicad_pcb (KiCad board)
At the start: 2 copper layers, 59 x 25 mm, 31 parts, among them J1 Conn_ARM_JTAG_SWD_10, J2 PWR_IN, M1 Fan_4pin, Q1 Q_NMOS_DGS, SW1 SW_Push, SW2 SW_Push, U2 STM32F042F6Px, U3 NCP1117-3.3_SOT223

Commit message: Various tweaks and adding more LEDs
Parts:
- removed R1, R2, R3, R4: 680r, Resistor_SMD:R_0603_1608Metric
- removed R10, R9: 10k, Resistor_SMD:R_0603_1608Metric
- removed SW2: SW_Push, Button_Switch_THT:SW_Tactile_SPST_Angled_PTS645Vx83-2LFS
- added D5: LED_Small, LED_THT:LED_D3.0mm_Horizontal_O1.27mm_Z2.0mm, F.Cu at (81.0, 72.0)
- added D6: LED_Small, LED_THT:LED_D3.0mm_Horizontal_O1.27mm_Z2.0mm, F.Cu at (86.0, 72.0)
- added D7: LED_Small, LED_THT:LED_D3.0mm_Horizontal_O1.27mm_Z2.0mm, F.Cu at (91.0, 72.0)
- added D8: LED_Small, LED_THT:LED_D3.0mm_Horizontal_O1.27mm_Z2.0mm, F.Cu at (96.0, 72.0)
- added IC1: NPIC6C596A, Package_SO:TSSOP-16_4.4x5mm_P0.65mm, F.Cu at (79.8, 66.5)
- added R11: 10k, Resistor_SMD:R_0603_1608Metric, F.Cu at (105.5, 66.2)
- added R12: 10k, Resistor_SMD:R_0603_1608Metric, F.Cu at (110.5, 66.2)
- added RN1: 680r, Resistor_SMD:R_Array_Convex_4x0612, F.Cu at (74.2, 66.5)
- added RN2: 680r, Resistor_SMD:R_Array_Convex_4x0612, F.Cu at (85.2, 66.5)
- SW1: value SW_Push -> RE111F-20B; footprint Button_Switch_THT:SW_Tactile_SPST_Angled_PTS645Vx83-2LFS -> pwmfan:RE111F-20B
- moved C5 18.5 mm to (89.0, 56.4), turned to 180 degrees
- moved R6 18.1 mm to (112.3, 59.3), turned to 90 degrees
- moved C2 18.0 mm to (92.8, 56.8), turned to 270 degrees
- moved R5 17.1 mm to (108.4, 60.1), turned to 180 degrees
- moved C1 16.9 mm to (103.8, 58.0)
- moved C3 16.9 mm to (103.8, 61.2)
- moved J1 16.9 mm to (100.4, 54.5)
- moved U2 16.9 mm to (97.8, 62.0)
- moved Q1 16.4 mm to (115.3, 61.1), turned to 270 degrees
- moved H2 16.0 mm to (120.0, 70.0)
- moved M1 15.9 mm to (120.9, 60.1)
- moved C4 14.7 mm to (89.0, 59.4), turned to 180 degrees
- moved SW1 11.0 mm to (108.0, 71.5), turned to 0 degrees
- moved D1 10.0 mm to (61.0, 72.0)
- moved D2 10.0 mm to (66.0, 72.0)
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Connections:
- U2 pad 10: SW_DOWN -> Net-(U2-Pad10)
- U2 pad 11: SW_UP -> ENC_A
- U2 pad 12: PWM -> ENC_B
- U2 pad 13: Net-(U2-Pad13) -> PWM
- U2 pad 6: Net-(R4-Pad2) -> SERIAL
- U2 pad 7: Net-(R3-Pad2) -> STORE_CLK
- U2 pad 8: Net-(R2-Pad2) -> SHIFT_CLK
Routing:
- net +3V3: track 108.1 -> 206.1 mm
- net STORE_CLK: track 0.00 -> 21.8 mm
- net SERIAL: track 0.00 -> 19.2 mm
- net SW_DOWN: track 19.2 -> 0.00 mm
- net SHIFT_CLK: track 0.00 -> 17.5 mm
- net ENC_B: track 0.00 -> 15.3 mm
- net SW_UP: track 15.2 -> 0.00 mm
- net Net-(D8-Pad1): track 0.00 -> 15.2 mm
- net Net-(D1-Pad1): track 2.31 -> 17.4 mm
- net +12V: track 57.8 -> 70.6 mm
- net Net-(R4-Pad2): track 12.8 -> 0.00 mm
- net ENC_A: track 0.00 -> 10.0 mm
- net Net-(U2-Pad9): track 9.60 -> 0.00 mm
- net Net-(D7-Pad1): track 0.00 -> 9.54 mm
- net Net-(D2-Pad1): track 2.31 -> 11.8 mm
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Other:
- board size 59 x 25 mm -> 75 x 25 mm

Commit message: Various updates and silks
Parts:
- removed D9: TS4148RXG, Diode_SMD:D_1206_3216Metric
- added Q2: DMG2307L, Package_TO_SOT_SMD:SOT-23, F.Cu at (72.0, 54.7)
- added R1: 10k, Resistor_SMD:R_0603_1608Metric, F.Cu at (98.6, 59.7)
- added R2: 10k, Resistor_SMD:R_0603_1608Metric, F.Cu at (101.6, 60.5)
- added R3: 3k3, Resistor_SMD:R_0603_1608Metric, F.Cu at (95.6, 60.5)
- added R4: PIN, Resistor_SMD:R_0603_1608Metric, F.Cu at (97.8, 62.7)
- added SYM1: QR, pwmfan:QR, B.Cu at (73.9, 58.9)
- Q1: value Q_NMOS_DGS -> BSS316N
- R5: value 0r -> BRD
- R6: value 100k -> 10k
- U3: value NCP1117-3.3_SOT223 -> NCP1117-3.3
- moved H2 27.0 mm to (97.5, 55.0)
- moved H1 16.8 mm to (62.5, 55.0)
- moved R12 15.1 mm to (95.4, 67.3)
- moved M1 14.9 mm to (106.0, 60.5)
- moved C1 13.2 mm to (91.0, 60.9)
- moved C3 13.1 mm to (91.0, 63.7)
- moved U2 13.0 mm to (85.0, 64.0)
- moved J1 12.9 mm to (87.5, 55.5)
- moved R11 11.8 mm to (93.8, 68.1)
- moved R6 11.6 mm to (102.2, 65.1)
- moved R5 11.4 mm to (97.8, 64.3)
- moved Q1 11.1 mm to (105.0, 65.2), turned to 0 degrees
- moved C2 10.6 mm to (82.5, 59.5), turned to 180 degrees
- moved C4 10.5 mm to (78.9, 62.4)
- moved C5 10.5 mm to (78.9, 59.4)
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Connections:
- F1 pad 1: +12V -> Net-(F1-Pad1)
- IC1 pad 9: Net-(IC1-Pad9) -> (no net)
- J1 pad 6: Net-(J1-Pad6) -> (no net)
- J1 pad 7: Net-(J1-Pad7) -> (no net)
- J1 pad 8: Net-(J1-Pad8) -> (no net)
- J2 pad 3: Net-(J2-Pad3) -> (no net)
- J2 pad 4: Net-(J2-Pad4) -> (no net)
- Q1 pad 1: Net-(M1-Pad1) -> Net-(Q1-Pad1)
- Q1 pad 2: Net-(Q1-Pad2) -> GND
- Q1 pad 3: GND -> Net-(M1-Pad1)
- R5 pad 1: Net-(Q1-Pad2) -> Net-(Q1-Pad1)
- R6 pad 1: Net-(Q1-Pad2) -> +3V3
- R6 pad 2: GND -> Net-(Q1-Pad1)
- U2 pad 1: Net-(U2-Pad1) -> (no net)
- U2 pad 10: Net-(U2-Pad10) -> (no net)
- U2 pad 14: Net-(U2-Pad14) -> TACHO
- U2 pad 17: Net-(U2-Pad17) -> (no net)
- U2 pad 18: Net-(U2-Pad18) -> (no net)
- U2 pad 2: Net-(U2-Pad2) -> (no net)
- U2 pad 3: Net-(U2-Pad3) -> (no net)
- U2 pad 9: Net-(U2-Pad9) -> (no net)
Routing:
- net +3V3: track 206.1 -> 173.7 mm
- net Net-(M1-Pad4): track 0.00 -> 15.3 mm
- net TACHO: track 0.00 -> 13.6 mm
- net Net-(M1-Pad3): track 0.00 -> 9.58 mm
- net Net-(F1-Pad2): track 5.69 -> 15.3 mm
- net Net-(Q1-Pad1): track 0.00 -> 5.36 mm
- net Net-(Q1-Pad2): track 5.16 -> 0.00 mm
- net +12V: track 70.6 -> 74.8 mm
- net SHIFT_CLK: track 17.5 -> 13.4 mm
- net SERIAL: track 19.2 -> 15.2 mm
- net STORE_CLK: track 21.8 -> 17.9 mm
- net PWM: track 9.47 -> 12.6 mm
- net Net-(F1-Pad1): track 0.00 -> 2.77 mm
- net Net-(D5-Pad1): track 8.48 -> 6.09 mm
- net ENC_A: track 10.0 -> 11.9 mm
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Other:
- board size 75 x 25 mm -> 60 x 25 mm
- net class Default: via_dia 0.8 -> 0.6; via_drill 0.4 -> 0.3
- net class PWR added: clearance 0.2, trace_width 1, via_dia 0.8, via_drill 0.4
- board text added: "PWMFan Thomas Bytheway 2020-02-25 Rev 1"

Commit message: Minor tweaks before shipping
Parts:
- RN1, RN2: value 680r -> 4x680r
Changed lines of the file:
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@@
     (34 B.Paste user)
     (35 F.Paste user)
-    (36 B.SilkS user hide)
+    (36 B.SilkS user)
     (37 F.SilkS user)
     (38 B.Mask user)
@@
       (effects (font (size 0.75 0.75) (thickness 0.12)))
     )
-    (fp_text value 680r (at -1.8 0 270) (layer F.SilkS)
+    (fp_text value 4x680r (at -1.8 0 270) (layer F.SilkS)
       (effects (font (size 0.75 0.75) (thickness 0.12)))
     )
@@
       (effects (font (size 0.75 0.75) (thickness 0.12)))
     )
-    (fp_text value 680r (at 1.8 0 270) (layer F.SilkS)
+    (fp_text value 4x680r (at 1.8 0 270) (layer F.SilkS)
       (effects (font (size 0.75 0.75) (thickness 0.12)))
     )
@@
       (effects (font (size 0.75 0.75) (thickness 0.12)))
     )
-    (fp_text value 10u (at 2.2 -0.4 180) (layer F.SilkS)
-      (effects (font (size 0.75 0.75) (thickness 0.12)))
-    )
+    (fp_text value 10u (at 2.2125 -0.05 180) (layer F.SilkS)
+      (effects (font (size 0.75 0.75) (thickness 0.12)))
+    )
